File: schematic/Thermometer.kicad_sch (KiCad schematic)
At the start: 16 parts, among them Q1 BC547, Q2 BC547, Q3 BC547, Q4 BC547, SW1 SW_SPDT, U1 CC56-12EWA, U2 DS18B20, U3 DS18B20

Commit message: Updated Readme Formatting and Schematic Comments
Other:
- note removed: "0"
- note removed: "30-03-2025"
- note removed: "Thermometer Diagram"
- title: (none) -> 7 Segment Thermometer
Changed lines of the file:
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@@
 	(generator_version "9.0")
 	(paper "A5")
-	(text "Thermometer Diagram"
-		(exclude_from_sim no)
-		(at 99.568 127.762 0)
-		(effects
-			(font
-				(size 1.27 1.27)
-			)
-			(justify left)
-		)
-	)
-	(text "30-03-2025"
-		(exclude_from_sim no)
-		(at 119.634 131.572 0)
-		(effects
-			(font
-				(size 1.27 1.27)
-			)
-			(justify left)
-		)
-	)
-	(text "0"
-		(exclude_from_sim no)
-		(at 181.356 131.572 0)
-		(effects
-			(font
-				(size 1.27 1.27)
-			)
-			(justify left)
-		)
+	(title_block
+		(title "7 Segment Thermometer")
+		(date "2025-03-30")
+		(rev "1.0")
 	)
 	(junction

Commit message: Optimized the display drawing routines and added optional serial temperature outputs
Parts:
- added R1: 1k, symbol Device:R_Small_US
Connections:
- net at A1.4 (GND), SW1.3 (C), U2.1 (GND)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: now also R1.2
- net at A1.22 (A3): now also R1.1
Changed lines of the file:
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@@
+	)
+	(junction
+		(at 54.61 95.25)
+		(diameter 0)
+		(color 0 0 0 0)
 	)
 	(junction
@@
 	(wire
 		(pts
+			(xy 52.07 76.2) (xy 54.61 76.2)
+		)
+		(stroke
+			(width 0)
+			(type default)
+		)
+	)
+	(wire
+		(pts
 			(xy 26.67 66.04) (xy 21.59 66.04)
 		)
@@
 	(wire
 		(pts
+			(xy 54.61 95.25) (xy 123.19 95.25)
+		)
+		(stroke
+			(width 0)
+			(type default)
+		)
+	)
+	(wire
+		(pts
 			(xy 25.4 21.59) (xy 26.67 21.59)
 		)
@@
 	(wire
 		(pts
-			(xy 39.37 95.25) (xy 123.19 95.25)
+			(xy 54.61 81.28) (xy 54.61 95.25)
+		)
+		(stroke
+			(width 0)
+			(type default)
+		)
+	)
+	(wire
+		(pts
+			(xy 39.37 95.25) (xy 54.61 95.25)
 		)
 		(stroke
@@
 					(unit 1)
 				)
+			)
+		)
+	)
+	(symbol
+		(lib_id "Device:R_Small_US")
+		(at 54.61 78.74 0)
+		(unit 1)
+		(exclude_from_sim no)
+		(in_bom yes)
+		(on_board yes)
+		(dnp no)
+		(fields_autoplaced yes)
+		(property "Reference" "R1"
+			(at 57.15 77.4699 0)
+			(effects
+				(font
+					(size 1.27 1.27)
+				)
+				(justify left)
+			)
+		)
+		(property "Value" "1k"
+			(at 57.15 80.0099 0)
+			(effects
+				(font
+					(size 1.27 1.27)
+				)
+				(justify left)
+			)
+		)
+		(property "Footprint" ""
+			(at 54.61 78.74 0)
+			(effects
+				(font
+					(size 1.27 1.27)
+				)
+				(hide yes)
+			)
+		)
+		(property "Datasheet" "~"
+			(at 54.61 78.74 0)
+			(effects
+				(font
+					(size 1.27 1.27)
+				)
+				(hide yes)
+			)
+		)
+		(property "Description" "Resistor, small US symbol"
+			(at 54.61 78.74 0)
+			(effects
+				(font
+					(size 1.27 1.27)
+				)
+				(hide yes)
+			)
+		)
+		(pin "1"
+		)
+		(pin "2"
+		)
+		(instances
+			(project ""
+				(path "/81b9514e-2b12-47cb-ad97-5183a669bf2a"
+					(reference "R1")
+					(unit 1)
+				)
